File: Circuit/Circuit.sch (KiCad schematic (older format))
At the start: 24 parts, among them J1 UE27AC54100, J2 22-23-2021, J3 22-23-2021, J4 22-23-2021, J5 22-23-2021, J6 22-23-2021, Q1 AO3401A, Q2 2N2222A, U1 L4978

Commit message: Finnished pcb design, and order PCB
Parts:
- added F1: Polyfuse, Fuse:Fuse_Bourns_MF-RHT300, symbol Device:Polyfuse
- added J7: 22-23-2021, Connector_PinHeader_2.54mm:PinHeader_1x02_P2.54mm_Vertical, symbol dk_Rectangular-Connectors-Headers-Male-Pins:22-23-2021
Connections:
- net +12V: now also F1.1; no longer C1.1, C7.1, R1.1, U1.5 (VCC)
- new net: C1.1, C7.1, F1.2, J7.1, J7.2, R1.1, U1.5 (VCC)
Other:
- moved on the sheet: J2
